File: power-expander/power-expander.kicad_pcb (KiCad board)
At the start: 2 copper layers, 50.5 x 55.5 mm, 12 parts, among them J1 Power, J2 Power, J3 Power, J4 Power, J5 Power, J6 Power, J7 Power, J8 Power

Commit message: Various improvements
Parts:
- added G***: LOGO, modular2:ibis-small, F.Cu at (93.0, 93.0)
Other:
- board text added: "POWER EXPANDER V2"
- board text removed: "POWER EXPANDER V1"
