File: envelope-generator/envelope-generator.kicad_pcb (KiCad board)
At the start: 2 copper layers, 60 x 80.2 mm, 35 parts, among them J1 Power, J2 Power, J3 Pot, J4 Pot, J5 Gate Input, J7 Output, SW1 Gate Button, SW2 AR/D Switch, U1 TL072

Commit message: Various improvements
Parts:
- moved R9 34.8 mm to (84.3, 100.0), turned to 0 degrees
- moved D6 27.1 mm to (100.2, 100.0)
- moved D2 17.9 mm to (110.3, 73.5), turned to 180 degrees
- moved R7 15.4 mm to (84.8, 95.0), turned to 0 degrees
- moved C2 12.3 mm to (97.0, 69.0)
- moved D5 11.5 mm to (96.5, 75.0), turned to 0 degrees
- moved J7 10.7 mm to (106.0, 82.0)
- moved J5 10.6 mm to (89.5, 82.0)
- moved R8 8.43 mm to (98.9, 95.0), turned to 0 degrees
- moved R2 3.58 mm to (100.5, 69.0)
- moved R6 2.42 mm to (97.6, 80.2), turned to -90 degrees
Routing:
- net GND: track 156.9 -> 179.5 mm
- net Net-(D5-A): track 9.35 -> 31.1 mm
- net Net-(D1-K): track 138.3 -> 149.6 mm
- net Net-(D6-A): track 18.8 -> 30.0 mm
- net Net-(J3-Pin_2): track 156.8 -> 166.2 mm
- net Net-(D2-K): track 3.92 -> 11.7 mm
- net Net-(D6-K): track 3.49 -> 11.0 mm
- net Net-(U1A-+): track 39.0 -> 31.5 mm
- net 12V: track 136.2 -> 143.1 mm
- net Net-(J7-Pin_1): track 16.7 -> 22.7 mm
- net Net-(C1-Pad2): track 42.8 -> 38.0 mm
- net Net-(U1A--): track 32.0 -> 33.9 mm
- net Net-(D1-A): track 27.9 -> 27.4 mm
Other:
- board text added: "ATK/REL"
- board text removed: "A/R"
