File: oscillator/oscillator.kicad_pcb (KiCad board)
At the start: 2 copper layers, 71 x 108 mm, 48 parts, among them J1 Power, J10 Conn_01x03_Socket, J2 Power, J3 Triangle Output, J4 Saw Output, J5 Pulse Output, J6 Frequency CV Input, J7 PWM CV Input, J8 Conn_01x03_Socket, J9 Conn_01x03_Socket, SW1 LFO Switch, U1 AS3340-custom, U2 TL074

Commit message: Various fixes
Parts:
- added J11: Power, Connector_IDC:IDC-Header_2x03_P2.54mm_Vertical, F.Cu at (100.5, 33.0)
- moved J1 34.7 mm to (64.5, 33.0)
- moved J2 16.8 mm to (82.5, 33.0)
- moved C1 7.63 mm to (82.5, 40.0), turned to 180 degrees
- moved R10 5.43 mm to (84.9, 40.0)
- moved R9 1.33 mm to (89.0, 53.0)
- moved R5 1.33 mm to (78.5, 42.9)
- moved R6 1.33 mm to (84.0, 42.9)
- moved R8 1.33 mm to (94.0, 53.1)
Routing:
- net -12V: track 124.8 -> 144.3 mm
- net GND: track 274.8 -> 267.0 mm
- net Net-(U1-VFCI): track 65.8 -> 71.5 mm
- net Net-(C1-Pad1): track 6.28 -> 2.42 mm
- net Net-(U2B-+): track 71.3 -> 67.4 mm
- net 12V: track 189.2 -> 193.0 mm
- net 5V: track 35.0 -> 38.2 mm
- net Net-(J9-Pin_2): track 25.8 -> 24.5 mm
- net Net-(J10-Pin_2): track 39.1 -> 38.5 mm
- net Net-(J6-Pin_1): track 16.1 -> 16.7 mm
- net Net-(J8-Pin_2): track 36.8 -> 36.3 mm

Commit message: Various improvements
Parts:
- added C7: 100nf, Capacitor_THT:C_Disc_D4.3mm_W1.9mm_P5.00mm, F.Cu at (105.0, 105.3)
- added C8: 100nf, Capacitor_THT:C_Disc_D4.3mm_W1.9mm_P5.00mm, F.Cu at (85.7, 106.0)
- added J12: Soft Sync, modular2:banana-jack, F.Cu at (96.5, 46.5)
- added J13: Hard Sync, modular2:banana-jack, F.Cu at (73.5, 46.5)
- moved C1 48.7 mm to (102.3, 84.5), turned to -90 degrees
- moved R5 13.4 mm to (65.1, 43.0)
- moved R8 11.0 mm to (105.0, 53.2)
- moved J7 5.57 mm to (56.5, 46.5)
- moved J6 5.50 mm to (113.5, 46.5)
- moved R10 4.30 mm to (88.0, 43.0), turned to -90 degrees
- moved R9 4.02 mm to (85.0, 53.2)
- moved R6 2.00 mm to (82.0, 43.0)
- moved C2 1.74 mm to (98.3, 89.5)
- moved C3 1.74 mm to (94.3, 89.5)
- moved C5 0.65 mm to (78.2, 106.0)
- moved R14 0.23 mm to (77.3, 129.2)
- moved R17 0.08 mm to (93.0, 119.0)
Connections:
- U1 pad 6: unconnected-(U1-VHSI-Pad6) -> Net-(U1-VHSI)
- U1 pad 9: unconnected-(U1-VSSI-Pad9) -> Net-(U1-VSSI)
Routing:
- net Net-(J12-Pin_1): track 0.00 -> 72.8 mm
- net Net-(J13-Pin_1): track 0.00 -> 67.0 mm
- net Net-(C1-Pad1): track 2.42 -> 47.4 mm
- net Net-(U2B-+): track 67.4 -> 80.9 mm
- net Net-(J7-Pin_1): track 51.1 -> 64.2 mm
- net Net-(J8-Pin_2): track 36.3 -> 24.9 mm
- net Net-(U1-VFCI): track 71.5 -> 80.8 mm
- net GND: track 267.0 -> 275.9 mm
- net Net-(J6-Pin_1): track 16.7 -> 11.2 mm
- net Net-(U1-VHSI): track 0.00 -> 4.17 mm
- net Net-(SW1-C): track 24.0 -> 28.1 mm
- net Net-(J10-Pin_2): track 38.5 -> 42.5 mm
- net Net-(SW1-A): track 13.8 -> 16.8 mm
- net Net-(U2B--): track 17.5 -> 14.6 mm
- net Net-(U1-VSSI): track 0.00 -> 2.87 mm
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Other:
- board text added: "HARD SYNC"
- board text added: "SOFT SYNC"
