File: note-sequencer/note-sequencer.kicad_pcb (KiCad board)
At the start: 2 copper layers, 157.4 x 181.1 mm, 95 parts, among them J1 Pitch, J2 Gate, J3 Velocity, J4 Clock, J5 Power, J6 Power, J7 Power, SW1 C1, SW10 A1, SW11 A#1, SW12 B1, SW13 C2, SW14 C#2, SW15 D2, SW16 D#2, SW17 E2, SW18 F2, SW19 F#2, SW2 C#1, SW20 G2, SW21 G#2, SW22 A2, SW23 A#2, SW24 B2, SW25 C3, SW26 X1, SW27 X2, SW28 X3, SW29 X4, SW3 D1, SW30 X5, SW31 RotaryEncoder_Switch, SW32 C2, SW33 Clock Source, SW34 SW_DIP_x01, SW35 Mode, SW4 D#1, SW5 E1, SW6 F1, SW7 F#1, SW8 G1, SW9 G#1, U4 TL072

Commit message: Update note sequencer
Parts:
- removed C4: 100nf, Capacitor_THT:C_Disc_D4.3mm_W1.9mm_P5.00mm
- added F0: foot, modular2:foot, B.Cu at (168.7, 19.8)
- added F1: foot, modular2:foot, B.Cu at (22.4, 19.8)
- added F2: foot, modular2:foot, B.Cu at (168.7, 190.4)
- added F3: foot, modular2:foot, B.Cu at (22.4, 190.4)
- added G***: LOGO, modular2:ibis-small, F.Cu at (96.0, 49.2)
- added J10: Gate, modular2:banana-jack, F.Cu at (57.8, 237.3)
- added J11: Velocity, modular2:banana-jack, F.Cu at (29.0, 264.6)
- added J12: Clock, modular2:banana-jack, F.Cu at (57.8, 264.6)
- added J13: LED Socket, Connector_PinHeader_2.54mm:PinHeader_1x02_P2.54mm_Vertical, F.Cu at (65.9, 246.1)
- added J14: Conn_01x06_Pin, Connector_PinHeader_2.54mm:PinHeader_1x06_P2.54mm_Vertical, F.Cu at (70.5, 242.5)
- added J6: Conn_01x06_Socket, Connector_PinSocket_2.54mm:PinSocket_1x06_P2.54mm_Vertical, F.Cu at (69.0, 42.8)
- added J9: Pitch, modular2:banana-jack, F.Cu at (29.0, 237.3)
- added REF**: MountingHole_3.2mm_M3, MountingHole:MountingHole_3.2mm_M3, F.Cu at (147.5, 167.5)
- added REF**: MountingHole_3.2mm_M3, MountingHole:MountingHole_3.2mm_M3, F.Cu at (157.5, 194.0)
- added REF**: MountingHole_3.2mm_M3, MountingHole:MountingHole_3.2mm_M3, F.Cu at (22.0, 230.1)
- added REF**: MountingHole_3.2mm_M3, MountingHole:MountingHole_3.2mm_M3, F.Cu at (24.5, 167.3)
- added REF**: MountingHole_3.2mm_M3, MountingHole:MountingHole_3.2mm_M3, F.Cu at (149.0, 367.1)
- added REF**: MountingHole_3.2mm_M3, MountingHole:MountingHole_3.2mm_M3, F.Cu at (69.0, 30.5)
- added REF**: MountingHole_3.2mm_M3, MountingHole:MountingHole_3.2mm_M3, F.Cu at (172.2, 275.4)
- added REF**: MountingHole_3.2mm_M3, MountingHole:MountingHole_3.2mm_M3, F.Cu at (26.0, 320.6)
- added REF**: MountingHole_3.2mm_M3, MountingHole:MountingHole_3.2mm_M3, F.Cu at (26.0, 366.9)
- added REF**: MountingHole_3.2mm_M3, MountingHole:MountingHole_3.2mm_M3, F.Cu at (77.8, 320.7)
- added REF**: MountingHole_3.2mm_M3, MountingHole:MountingHole_3.2mm_M3, F.Cu at (33.5, 194.0)
- added REF**: MountingHole_3.2mm_M3, MountingHole:MountingHole_3.2mm_M3, F.Cu at (70.5, 274.1)
- added REF**: MountingHole_3.2mm_M3, MountingHole:MountingHole_3.2mm_M3, F.Cu at (76.3, 121.0)
- added REF**: MountingHole_3.2mm_M3, MountingHole:MountingHole_3.2mm_M3, F.Cu at (70.5, 230.1)
- added REF**: MountingHole_3.2mm_M3, MountingHole:MountingHole_3.2mm_M3, F.Cu at (97.2, 393.6)
- added REF**: MountingHole_3.2mm_M3, MountingHole:MountingHole_3.2mm_M3, F.Cu at (77.8, 367.1)
- added REF**: MountingHole_3.2mm_M3, MountingHole:MountingHole_3.2mm_M3, F.Cu at (20.5, 30.5)
- added REF**: MountingHole_3.2mm_M3, MountingHole:MountingHole_3.2mm_M3, F.Cu at (147.5, 121.0)
- added REF**: MountingHole_3.2mm_M3, MountingHole:MountingHole_3.2mm_M3, F.Cu at (35.0, 393.6)
- added REF**: MountingHole_3.2mm_M3, MountingHole:MountingHole_3.2mm_M3, F.Cu at (76.3, 167.5)
- added REF**: MountingHole_3.2mm_M3, MountingHole:MountingHole_3.2mm_M3, F.Cu at (170.7, 75.8)
- added REF**: MountingHole_3.2mm_M3, MountingHole:MountingHole_3.2mm_M3, F.Cu at (95.7, 194.0)
- added REF**: MountingHole_3.2mm_M3, MountingHole:MountingHole_3.2mm_M3, F.Cu at (69.0, 74.5)
- added REF**: MountingHole_3.2mm_M3, MountingHole:MountingHole_3.2mm_M3, F.Cu at (24.5, 121.0)
- added REF**: MountingHole_3.2mm_M3, MountingHole:MountingHole_3.2mm_M3, F.Cu at (149.0, 320.6)
- added REF**: MountingHole_3.2mm_M3, MountingHole:MountingHole_3.2mm_M3, F.Cu at (159.0, 393.6)
- moved J5 35.8 mm to (141.9, 19.5)
- moved SW1 27.2 mm to (163.8, 48.6)
- moved J4 15.0 mm to (93.1, 19.5)
- moved D1 9.37 mm to (56.3, 48.7), turned to 90 degrees
- moved D21 8.85 mm to (31.7, 189.2)
- moved R2 8.50 mm to (22.3, 51.0)
- moved R1 7.50 mm to (22.3, 47.5)
- moved J3 6.73 mm to (44.0, 19.5)
- moved D32 6.66 mm to (151.7, 189.2)
- moved RV2 6.25 mm to (54.0, 55.5)
- moved RV1 6.25 mm to (25.0, 55.5)
- moved U3 5.52 mm to (81.8, 41.7)
- moved A1 5.21 mm to (130.6, 43.8)
- moved A2 5.21 mm to (130.6, 68.6)
- moved C3 5.21 mm to (133.2, 50.0)
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- renumbered A2 to A1, A1 to A2, C6 to C1, C5 to C2, C2 to C3, D32 to D1, D7 to D10, D1 to D12, D3 to D13, D5 to D14, D6 to D15, D8 to D16, D12 to D17, D10 to D18, D13 to D19, D26 to D2, D14 to D20, D31 to D21, D16 to D22, D15 to D23, D17 to D24, D18 to D25, D21 to D26, D20 to D27, D19 to D28, D23 to D29, D28 to D3, D22 to D30, D24 to D31, D25 to D32, D27 to D4, D29 to D5, D30 to D6, D2 to D7, D4 to D8, J5 to J3, J6 to J4, J7 to J5, J3 to J7, J4 to J8, R5 to R1, R6 to R2, R7 to R5, R9 to R6, R8 to R7, R1 to R8, R2 to R9, SW34 to SW1, SW4 to SW10, SW2 to SW11, SW7 to SW12, SW11 to SW13, SW9 to SW14, SW1 to SW15, SW3 to SW16, SW5 to SW17, SW6 to SW18, SW8 to SW19, SW26 to SW2, SW10 to SW20, SW12 to SW21, SW13 to SW22, SW14 to SW23, SW16 to SW24, SW19 to SW25, SW21 to SW26, SW23 to SW27, SW32 to SW28, SW15 to SW29, SW27 to SW3, SW18 to SW30, SW17 to SW31, SW20 to SW32, SW22 to SW33, SW24 to SW34, SW25 to SW35, SW28 to SW4, SW29 to SW5, SW30 to SW6, SW31 to SW7, SW33 to SW8, SW35 to SW9, U2 to U1, U4 to U2, U1 to U3, U3 to U4
Routing:
- net GND: track 241.5 -> 369.3 mm
- net 12V: track 43.8 -> 151.4 mm
- net 5V: track 98.7 -> 200.7 mm
- net -12V: track 38.8 -> 136.1 mm
- net Net-(A2-D11): track 6.49 -> 97.9 mm
- net Net-(A2-D10): track 5.92 -> 96.1 mm
- net Net-(A2-D9): track 5.36 -> 94.3 mm
- net Net-(J1-Pin_1): track 16.9 -> 104.6 mm
- net Net-(A2-D8): track 4.79 -> 92.5 mm
- net Net-(A2-D13): track 14.5 -> 96.7 mm
- net Net-(A2-3V3): track 13.9 -> 92.0 mm
- net Net-(J3-Pin_1): track 10.1 -> 85.8 mm
- net Net-(A2-D2): track 4.22 -> 79.0 mm
- net Net-(J10-Pin_1): track 0.00 -> 54.9 mm
- net Net-(J11-Pin_1): track 0.00 -> 47.2 mm
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Other:
- board size 157.4 x 181.1 mm -> 160.9 x 383.9 mm
- board text added: "NOTE SEQUENCER V1"

Commit message: Updates
Parts:
- removed C3: 100nf, Capacitor_THT:C_Disc_D4.3mm_W1.9mm_P5.00mm
- added C2: 100nf, Capacitor_THT:C_Disc_D4.3mm_W1.9mm_P5.00mm, F.Cu at (140.5, 50.0)
- added SW30: SW_DIP_x01, Button_Switch_THT:SW_DIP_SPSTx01_Slide_9.78x4.72mm_W7.62mm_P2.54mm, F.Cu at (127.9, 48.6)
- moved R1 6.92 mm to (158.1, 50.0)
- moved R2 6.92 mm to (158.1, 47.0)
- renumbered A2 to A1, A1 to A2, C2 to C5, C1 to C6, D12 to D1, D18 to D10, D17 to D12, D19 to D13, D20 to D14, D23 to D15, D22 to D16, D24 to D17, D25 to D18, D28 to D19, D7 to D2, D27 to D20, D26 to D21, D30 to D22, D29 to D23, D31 to D24, D32 to D25, D2 to D26, D4 to D27, D3 to D28, D5 to D29, D13 to D3, D6 to D30, D21 to D31, D1 to D32, D8 to D4, D14 to D5, D15 to D6, D10 to D7, D16 to D8, J11 to J10, J9 to J11, J10 to J13, J13 to J14, J7 to J3, J8 to J4, J3 to J5, J4 to J6, J5 to J7, J6 to J8, J14 to J9, R8 to R1, R9 to R2, R1 to R5, R2 to R6, R5 to R7, R7 to R8, R6 to R9, SW15 to SW1, SW20 to SW10, SW13 to SW11, SW21 to SW12, SW22 to SW13, SW23 to SW14, SW29 to SW15, SW24 to SW16, SW31 to SW17, SW30 to SW18, SW25 to SW19, SW11 to SW2, SW32 to SW20, SW26 to SW21, SW33 to SW22, SW27 to SW23, SW34 to SW24, SW35 to SW25, SW2 to SW26, SW3 to SW27, SW4 to SW28, SW5 to SW29, SW16 to SW3, SW7 to SW31, SW28 to SW32, SW8 to SW33, SW1 to SW34, SW9 to SW35, SW10 to SW4, SW17 to SW5, SW18 to SW6, SW12 to SW7, SW19 to SW8, SW14 to SW9, U3 to U1, U1 to U2, U4 to U3, U2 to U4
Connections:
- U1 pad 11: Net-(A2-D2) -> Net-(U1-Lite)
Routing:
- net Net-(A2-D2): track 79.0 -> 7.23 mm
- net Net-(U1-Lite): track 0.00 -> 57.5 mm
- net Net-(A1-A5): track 180.5 -> 191.7 mm
- net GND: track 369.3 -> 378.0 mm
- net 5V: track 200.7 -> 209.2 mm
- net Net-(A1-A4): track 177.9 -> 184.2 mm

Commit message: Fix issue with extra button
Parts:
- removed the SW6 at (107.9, 82.9)
- moved D30 57.7 mm to (157.0, 84.9), turned to -90 degrees
Routing:
- net Net-(A1-D12): track 456.9 -> 387.0 mm
- net Net-(D30-A): track 57.8 -> 6.75 mm
- net Net-(A1-D2): track 157.1 -> 170.2 mm

Commit message: More fixes
Parts:
- R6: renamed from R9; value 10K -> 1K
- renumbered A2 to A1, A1 to A2, C6 to C1, C5 to C2, C2 to C3, D32 to D1, D9 to D10, D1 to D12, D3 to D13, D5 to D14, D6 to D15, D8 to D16, D10 to D17, D12 to D18, D13 to D19, D30 to D2, D14 to D20, D31 to D21, D17 to D22, D16 to D23, D15 to D24, D18 to D25, D19 to D26, D21 to D27, D20 to D28, D22 to D29, D26 to D3, D23 to D30, D24 to D31, D25 to D32, D28 to D4, D27 to D5, D29 to D6, D2 to D7, D4 to D8, D7 to D9, J13 to J10, J10 to J11, J14 to J13, J9 to J14, J5 to J3, J6 to J4, J7 to J5, J8 to J6, J3 to J7, J4 to J8, J11 to J9, R3 to R1, R5 to R2, R6 to R3, R8 to R5, R1 to R8, R2 to R9, SW30 to SW1, SW2 to SW10, SW4 to SW11, SW7 to SW12, SW9 to SW13, SW11 to SW14, SW1 to SW15, SW3 to SW16, SW6 to SW17, SW5 to SW18, SW8 to SW19, SW34 to SW2, SW10 to SW20, SW12 to SW21, SW13 to SW22, SW14 to SW23, SW16 to SW24, SW19 to SW25, SW21 to SW26, SW23 to SW27, SW32 to SW28, SW15 to SW29, SW26 to SW3, SW17 to SW30, SW18 to SW31, SW20 to SW32, SW22 to SW33, SW24 to SW34, SW25 to SW35, SW27 to SW4, SW29 to SW5, SW28 to SW6, SW31 to SW7, SW35 to SW8, SW33 to SW9, U4 to U1, U1 to U3, U3 to U4
Other:
- outline, holes or cut-outs redrawn
