File: gate-sequencer/gate-sequencer.kicad_pcb (KiCad board)
At the start: 2 copper layers, 109 parts, among them J1 Gate 8, J10 Gate 6, J11 Gate 10, J12 Gate 14, J13 Gate 1, J14 Gate 5, J15 Gate 9, J16 Gate 13, J2 Gate 4, J3 Gate 12, J4 Gate 16, J5 Gate 3, J6 Gate 7, J7 Gate 11, J8 Gate 15, J9 Gate 2, SW1 X1, SW10 S6, SW11 S7, SW12 S8, SW13 S9, SW14 S10, SW15 S11, SW16 S12, SW17 S13, SW18 S14, SW19 S15, SW2 X2, SW20 S16, SW3 X3, SW35 Mode, SW4 X4, SW5 S1, SW6 S2, SW7 S3, SW8 S4, SW9 S5

Commit message: Progress gate sequencer
Parts:
- moved J4 210.6 mm to (232.8, 110.8)
- moved J1 210.4 mm to (231.6, 60.8)
- moved J6 180.4 mm to (212.3, 60.8)
- moved SW12 179.0 mm to (234.1, 83.5)
- moved J8 178.2 mm to (213.3, 110.8)
- moved SW20 163.1 mm to (234.1, 133.5)
- moved SW11 162.3 mm to (214.9, 83.5)
- moved SW19 153.6 mm to (214.9, 133.5)
- moved J10 148.8 mm to (193.1, 60.8)
- moved D20 148.4 mm to (237.1, 119.7), turned to -90 degrees
- moved SW10 147.9 mm to (195.6, 83.5)
- moved SW18 147.6 mm to (195.6, 133.5)
- moved R7 147.2 mm to (234.5, 127.3), turned to 180 degrees
- moved J12 145.7 mm to (193.9, 110.8)
- moved R3 145.6 mm to (234.5, 77.3), turned to 180 degrees
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Routing:
- net GND: track 0.00 -> 330.1 mm
- net Net-(D1-K): track 0.00 -> 282.7 mm
- net Net-(D10-K): track 0.00 -> 266.0 mm
- net Net-(D11-K): track 0.00 -> 260.0 mm
- net Net-(D12-K): track 0.00 -> 246.0 mm
- net Net-(SW13-Pad2): track 0.00 -> 151.6 mm
- net Net-(SW5-Pad2): track 0.00 -> 151.4 mm
- net Net-(U1-S7): track 0.00 -> 144.9 mm
- net Net-(U1-S15): track 0.00 -> 142.7 mm
- net Net-(U1-S6): track 0.00 -> 126.2 mm
- net Net-(U1-S14): track 0.00 -> 123.4 mm
- net Net-(U1-S5): track 0.00 -> 106.7 mm
- net Net-(U1-S13): track 0.00 -> 103.9 mm
- net Net-(J10-Pin_1): track 0.00 -> 103.1 mm
- net Net-(J13-Pin_1): track 0.00 -> 103.0 mm
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
Commit message: Updates
Parts:
- removed C1: 100nf, Capacitor_THT:C_Disc_D4.3mm_W1.9mm_P5.00mm
- added C3: 100nf, Capacitor_THT:C_Disc_D4.3mm_W1.9mm_P5.00mm, F.Cu at (178.0, 43.8)
- added G***: LOGO, modular2:ibis-small, F.Cu at (119.5, 55.0)
- added J17: Clock, modular2:banana-jack, F.Cu at (171.0, 31.0)
- added J18: Conn_01x34_Socket, Connector_PinSocket_2.54mm:PinSocket_1x34_P2.54mm_Vertical, F.Cu at (61.2, 173.5)
- added J19: Power, Connector_IDC:IDC-Header_2x03_P2.54mm_Vertical, F.Cu at (50.9, 14.0)
- added J20: Power, Connector_IDC:IDC-Header_2x03_P2.54mm_Vertical, F.Cu at (99.1, 14.0)
- added J21: Power, Connector_IDC:IDC-Header_2x03_P2.54mm_Vertical, F.Cu at (147.3, 14.0)
- added J22: Clock, modular2:banana-jack, F.Cu at (354.0, 27.5)
- added J23: Gate 1, modular2:banana-jack, F.Cu at (217.2, 79.3)
- added J24: Gate 9, modular2:banana-jack, F.Cu at (217.2, 129.4)
- added J25: Gate 2, modular2:banana-jack, F.Cu at (236.5, 79.3)
- added J26: Gate 10, modular2:banana-jack, F.Cu at (236.7, 129.4)
- added J27: Gate 3, modular2:banana-jack, F.Cu at (255.7, 79.3)
- added J28: Gate 11, modular2:banana-jack, F.Cu at (256.1, 129.4)
- added J29: Gate 4, modular2:banana-jack, F.Cu at (275.0, 79.3)
- added J30: Gate 12, modular2:banana-jack, F.Cu at (275.6, 129.4)
- added J31: Gate 5, modular2:banana-jack, F.Cu at (294.3, 79.3)
- added J32: Gate 13, modular2:banana-jack, F.Cu at (295.0, 129.4)
- added J33: Gate 6, modular2:banana-jack, F.Cu at (313.5, 79.3)
- added J34: Gate 14, modular2:banana-jack, F.Cu at (314.4, 129.4)
- added J35: Gate 7, modular2:banana-jack, F.Cu at (332.8, 79.3)
- added J36: Gate 15, modular2:banana-jack, F.Cu at (333.9, 129.4)
- added J37: Gate 8, modular2:banana-jack, F.Cu at (352.1, 79.3)
- added J38: Gate 16, modular2:banana-jack, F.Cu at (353.3, 129.4)
- added J39: LED, Connector_PinHeader_2.54mm:PinHeader_1x02_P2.54mm_Vertical, F.Cu at (210.0, 89.3)
- added J40: LED, Connector_PinHeader_2.54mm:PinHeader_1x02_P2.54mm_Vertical, F.Cu at (209.8, 139.3)
- added J41: LED, Connector_PinHeader_2.54mm:PinHeader_1x02_P2.54mm_Vertical, F.Cu at (229.2, 89.3)
- added J42: LED, Connector_PinHeader_2.54mm:PinHeader_1x02_P2.54mm_Vertical, F.Cu at (229.0, 139.3)
- added J43: LED, Connector_PinHeader_2.54mm:PinHeader_1x02_P2.54mm_Vertical, F.Cu at (248.4, 89.3)
- added J44: LED, Connector_PinHeader_2.54mm:PinHeader_1x02_P2.54mm_Vertical, F.Cu at (248.2, 139.3)
- added J45: LED, Connector_PinHeader_2.54mm:PinHeader_1x02_P2.54mm_Vertical, F.Cu at (267.6, 89.3)
- added J46: LED, Connector_PinHeader_2.54mm:PinHeader_1x02_P2.54mm_Vertical, F.Cu at (267.5, 139.3)
- added J47: LED, Connector_PinHeader_2.54mm:PinHeader_1x02_P2.54mm_Vertical, F.Cu at (286.8, 89.3)
- added J48: LED, Connector_PinHeader_2.54mm:PinHeader_1x02_P2.54mm_Vertical, F.Cu at (286.7, 139.3)
- added J49: LED, Connector_PinHeader_2.54mm:PinHeader_1x02_P2.54mm_Vertical, F.Cu at (306.0, 89.3)
- added J50: LED, Connector_PinHeader_2.54mm:PinHeader_1x02_P2.54mm_Vertical, F.Cu at (306.0, 139.3)
- added J51: LED, Connector_PinHeader_2.54mm:PinHeader_1x02_P2.54mm_Vertical, F.Cu at (325.2, 89.3)
- added J52: LED, Connector_PinHeader_2.54mm:PinHeader_1x02_P2.54mm_Vertical, F.Cu at (325.2, 139.3)
- added J53: LED, Connector_PinHeader_2.54mm:PinHeader_1x02_P2.54mm_Vertical, F.Cu at (344.4, 89.3)
- added J54: LED, Connector_PinHeader_2.54mm:PinHeader_1x02_P2.54mm_Vertical, F.Cu at (344.4, 139.3)
- added J55: Conn_01x34_Pin, Connector_PinHeader_2.54mm:PinHeader_1x34_P2.54mm_Vertical, F.Cu at (244.1, 170.0)
- added R33: 1K, Resistor_THT:R_Axial_DIN0207_L6.3mm_D2.5mm_P10.16mm_Horizontal, F.Cu at (162.9, 36.0)
- added REF**: MountingHole_3.2mm_M3, MountingHole:MountingHole_3.2mm_M3, F.Cu at (22.5, 23.0)
- added REF**: MountingHole_3.2mm_M3, MountingHole:MountingHole_3.2mm_M3, F.Cu at (364.0, 173.5)
- added REF**: MountingHole_3.2mm_M3, MountingHole:MountingHole_3.2mm_M3, F.Cu at (77.6, 69.5)
- added REF**: MountingHole_3.2mm_M3, MountingHole:MountingHole_3.2mm_M3, F.Cu at (205.5, 172.5)
- added REF**: MountingHole_3.2mm_M3, MountingHole:MountingHole_3.2mm_M3, F.Cu at (125.7, 69.5)
- added REF**: MountingHole_3.2mm_M3, MountingHole:MountingHole_3.2mm_M3, F.Cu at (285.2, 123.5)
- added REF**: MountingHole_3.2mm_M3, MountingHole:MountingHole_3.2mm_M3, F.Cu at (181.0, 38.5)
- added REF**: MountingHole_3.2mm_M3, MountingHole:MountingHole_3.2mm_M3, F.Cu at (181.0, 177.0)
- added REF**: MountingHole_3.2mm_M3, MountingHole:MountingHole_3.2mm_M3, F.Cu at (364.0, 66.0)
- added REF**: MountingHole_3.2mm_M3, MountingHole:MountingHole_3.2mm_M3, F.Cu at (260.6, 66.0)
- added REF**: MountingHole_3.2mm_M3, MountingHole:MountingHole_3.2mm_M3, F.Cu at (102.2, 127.0)
- added REF**: MountingHole_3.2mm_M3, MountingHole:MountingHole_3.2mm_M3, F.Cu at (181.0, 69.5)
- added REF**: MountingHole_3.2mm_M3, MountingHole:MountingHole_3.2mm_M3, F.Cu at (205.5, 19.5)
- added REF**: MountingHole_3.2mm_M3, MountingHole:MountingHole_3.2mm_M3, F.Cu at (308.7, 66.0)
- added REF**: MountingHole_3.2mm_M3, MountingHole:MountingHole_3.2mm_M3, F.Cu at (22.5, 176.0)
- added REF**: MountingHole_3.2mm_M3, MountingHole:MountingHole_3.2mm_M3, F.Cu at (364.0, 35.0)
- added REF**: MountingHole_3.2mm_M3, MountingHole:MountingHole_3.2mm_M3, F.Cu at (364.0, 19.5)
- added REF**: MountingHole_3.2mm_M3, MountingHole:MountingHole_3.2mm_M3, F.Cu at (181.0, 23.0)
- added RV1: 100K - Tempo, Potentiometer_THT:Potentiometer_Alps_RK09K_Single_Vertical, F.Cu at (70.2, 37.0)
- added RV2: 100K - Period, Potentiometer_THT:Potentiometer_Alps_RK09K_Single_Vertical, F.Cu at (31.7, 37.0)
- added SW21: Mode, modular2:switch1, F.Cu at (128.0, 31.0)
- added SW22: Mode 2, modular2:switch1, F.Cu at (113.0, 31.0)
- SW35: value Mode -> Clock Source
- moved D10 66.3 mm to (136.1, 91.7)
- moved D13 66.3 mm to (39.7, 141.7)
- moved D19 66.3 mm to (155.3, 141.7)
- moved D23 66.3 mm to (167.9, 144.0)
- moved D27 66.3 mm to (148.6, 144.0)
- moved D30 66.3 mm to (52.0, 144.0)
- moved D35 66.3 mm to (32.7, 144.0)
- moved J12 66.3 mm to (131.4, 132.7)
- moved J3 66.3 mm to (92.5, 132.7)
- moved R11 66.3 mm to (143.2, 86.1)
- moved R17 66.3 mm to (46.4, 86.1)
- moved R18 66.3 mm to (56.4, 99.3)
- moved R20 66.3 mm to (133.5, 99.3)
- moved R23 66.3 mm to (123.2, 136.1)
- moved R24 66.3 mm to (133.4, 149.2)
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Connections:
- A1 pad 1: unconnected-(A1-D1/TX-Pad1) -> Net-(A1-D1/TX)
- A1 pad 10: unconnected-(A1-D7-Pad10) -> Net-(A1-D7)
- A1 pad 11: unconnected-(A1-D8-Pad11) -> Net-(A1-D8)
- A1 pad 12: unconnected-(A1-D9-Pad12) -> Net-(A1-D9)
- A1 pad 13: unconnected-(A1-D10-Pad13) -> Net-(A1-D10)
- A1 pad 14: unconnected-(A1-D11-Pad14) -> Net-(A1-D11)
- A1 pad 15: unconnected-(A1-D12-Pad15) -> Net-(A1-D12)
- A1 pad 18: unconnected-(A1-AREF-Pad18) -> Net-(A1-AREF)
- A1 pad 19: unconnected-(A1-A0-Pad19) -> Net-(A1-A0)
- A1 pad 2: unconnected-(A1-D0/RX-Pad2) -> Net-(A1-D0/RX)
- A1 pad 20: unconnected-(A1-A1-Pad20) -> Net-(A1-A1)
- A1 pad 21: unconnected-(A1-A2-Pad21) -> Net-(A1-A2)
- A1 pad 22: unconnected-(A1-A3-Pad22) -> Net-(A1-A3)
- A1 pad 23: unconnected-(A1-A4-Pad23) -> Net-(A1-A4)
- A1 pad 24: unconnected-(A1-A5-Pad24) -> Net-(A1-A5)
- A1 pad 25: unconnected-(A1-A6-Pad25) -> Net-(A1-A6)
- A1 pad 26: unconnected-(A1-A7-Pad26) -> Net-(A1-A7)
- A1 pad 5: unconnected-(A1-D2-Pad5) -> Net-(A1-D2)
- A1 pad 6: unconnected-(A1-D3-Pad6) -> Net-(A1-D3)
- A1 pad 7: unconnected-(A1-D4-Pad7) -> Net-(A1-D4)
- A1 pad 8: unconnected-(A1-D5-Pad8) -> Net-(A1-D5)
- A1 pad 9: unconnected-(A1-D6-Pad9) -> Net-(A1-D6)
- D1 pad 1: Net-(D1-K) -> Net-(A1-D8)
- D10 pad 1: Net-(D10-K) -> Net-(A1-D9)
- D11 pad 1: Net-(D11-K) -> Net-(A1-D10)
- D12 pad 1: Net-(D12-K) -> Net-(A1-D11)
- D13 pad 1: Net-(D1-K) -> Net-(A1-D8)
- D14 pad 1: Net-(D10-K) -> Net-(A1-D9)
- D15 pad 1: Net-(D11-K) -> Net-(A1-D10)
- D16 pad 1: Net-(D12-K) -> Net-(A1-D11)
- D17 pad 1: Net-(D1-K) -> Net-(A1-D8)
- D18 pad 1: Net-(D10-K) -> Net-(A1-D9)
- D19 pad 1: Net-(D11-K) -> Net-(A1-D10)
- D2 pad 1: Net-(D10-K) -> Net-(A1-D9)
- D20 pad 1: Net-(D12-K) -> Net-(A1-D11)
- D3 pad 1: Net-(D11-K) -> Net-(A1-D10)
- D4 pad 1: Net-(D12-K) -> Net-(A1-D11)
- D5 pad 1: Net-(D1-K) -> Net-(A1-D8)
- D6 pad 1: Net-(D10-K) -> Net-(A1-D9)
- D7 pad 1: Net-(D11-K) -> Net-(A1-D10)
- D8 pad 1: Net-(D12-K) -> Net-(A1-D11)
- D9 pad 1: Net-(D1-K) -> Net-(A1-D8)
- SW1 pad 2: Net-(SW1-Pad2) -> Net-(A1-D7)
- SW10 pad 2: Net-(SW10-Pad2) -> Net-(A1-D5)
- SW11 pad 2: Net-(SW10-Pad2) -> Net-(A1-D5)
- SW12 pad 2: Net-(SW10-Pad2) -> Net-(A1-D5)
- SW13 pad 2: Net-(SW13-Pad2) -> Net-(A1-D4)
- SW14 pad 2: Net-(SW13-Pad2) -> Net-(A1-D4)
- SW15 pad 2: Net-(SW13-Pad2) -> Net-(A1-D4)
- SW16 pad 2: Net-(SW13-Pad2) -> Net-(A1-D4)
- SW17 pad 2: Net-(SW17-Pad2) -> Net-(A1-D3)
- SW18 pad 2: Net-(SW17-Pad2) -> Net-(A1-D3)
- SW19 pad 2: Net-(SW17-Pad2) -> Net-(A1-D3)
- SW2 pad 2: Net-(SW1-Pad2) -> Net-(A1-D7)
- SW20 pad 2: Net-(SW17-Pad2) -> Net-(A1-D3)
- SW3 pad 2: Net-(SW1-Pad2) -> Net-(A1-D7)
- SW35 pad 2: unconnected-(SW35-B-Pad2) -> Net-(A1-D0/RX)
- SW35 pad 3: unconnected-(SW35-A-Pad3) -> GND
- SW4 pad 2: Net-(SW1-Pad2) -> Net-(A1-D7)
- SW5 pad 2: Net-(SW5-Pad2) -> Net-(A1-D6)
- SW6 pad 2: Net-(SW5-Pad2) -> Net-(A1-D6)
- SW7 pad 2: Net-(SW5-Pad2) -> Net-(A1-D6)
- SW8 pad 2: Net-(SW5-Pad2) -> Net-(A1-D6)
- SW9 pad 2: Net-(SW10-Pad2) -> Net-(A1-D5)
- U1 pad 1: unconnected-(U1-STROBE-Pad1) -> Net-(A1-A5)
- U1 pad 2: unconnected-(U1-A-Pad2) -> Net-(A1-A0)
- U1 pad 21: unconnected-(U1-C-Pad21) -> Net-(A1-A2)
- U1 pad 22: unconnected-(U1-D-Pad22) -> Net-(A1-A3)
- U1 pad 23: unconnected-(U1-INHIBIT-Pad23) -> Net-(A1-A4)
- U1 pad 3: unconnected-(U1-B-Pad3) -> Net-(A1-A1)
Routing:
- net GND: track 330.1 -> 1060.7 mm
- net Net-(J39-Pin_2): track 0.00 -> 442.5 mm
- net 5V: track 0.00 -> 396.5 mm
- net Net-(J22-Pin_1): track 0.00 -> 381.2 mm
- net Net-(A1-D8): track 0.00 -> 308.8 mm
- net Net-(D1-K): track 282.7 -> 0.00 mm
- net Net-(A1-D9): track 0.00 -> 279.8 mm
- net Net-(A1-D10): track 0.00 -> 273.3 mm
- net Net-(D10-K): track 266.0 -> 0.00 mm
- net Net-(J45-Pin_1): track 0.00 -> 262.4 mm
- net Net-(D11-K): track 260.0 -> 0.00 mm
- net Net-(J47-Pin_1): track 0.00 -> 255.1 mm
- net Net-(A1-D4): track 0.00 -> 254.7 mm
- net Net-(A1-D11): track 0.00 -> 249.3 mm
- net Net-(J31-Pin_1): track 0.00 -> 247.8 mm
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Other:
- board outline added: 349.3 x 174.9 mm
- board text added: "GATE SEQUENCER V1"

Commit message: Renumber some components
Parts:
- moved J25 259.6 mm to (70.6, 261.2)
- moved J26 259.6 mm to (109.1, 261.2)
- moved J29 259.6 mm to (147.6, 261.2)
- moved J31 259.6 mm to (24.8, 271.2)
- moved J32 259.6 mm to (63.2, 271.2)
- moved J33 259.6 mm to (44.0, 271.2)
- moved J34 259.6 mm to (82.4, 271.2)
- moved J35 259.6 mm to (101.6, 271.2)
- moved J36 259.6 mm to (120.8, 271.2)
- moved J37 259.6 mm to (159.3, 271.2)
- moved J38 259.6 mm to (140.1, 271.2)
- moved J40 259.6 mm to (51.5, 311.3)
- moved J41 259.6 mm to (70.9, 311.3)
- moved J42 259.6 mm to (109.8, 311.3)
- moved J44 259.6 mm to (129.2, 311.3)
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- renumbered C2 to C1, C3 to C2, D2 to D1, D24 to D10, D8 to D11, D32 to D12, D34 to D13, D9 to D14, D29 to D15, D10 to D16, D11 to D17, D25 to D18, D21 to D19, D1 to D2, D12 to D20, D35 to D21, D13 to D22, D14 to D23, D30 to D24, D26 to D25, D15 to D26, D16 to D27, D36 to D28, D22 to D29, D18 to D30, D17 to D32, D27 to D33, D19 to D34, D23 to D35, D20 to D36, D33 to D5, D28 to D6, D6 to D7, D5 to D8, D7 to D9, J19 to J1, J6 to J11, J1 to J12, J15 to J13, J11 to J14, J7 to J15, J3 to J16, J16 to J17, J12 to J18, J8 to J19, J20 to J2, J4 to J20, J18 to J21, J25 to J24, J27 to J25, J31 to J26, J29 to J27, J33 to J28, J35 to J29, J21 to J3, J37 to J30, J39 to J31, J43 to J32, J41 to J33, J45 to J34, J47 to J35, J49 to J36, J53 to J37, J51 to J38, J24 to J39, J17 to J4, J26 to J40, J28 to J41, J32 to J42, J30 to J43, J34 to J44, J36 to J45, J38 to J46, J40 to J47, J44 to J48, J42 to J49, J13 to J5, J46 to J50, J48 to J51, J50 to J52, J52 to J53, J9 to J6, J5 to J7, J2 to J8, J14 to J9, R33 to R1, R26 to R10, R18 to R11, R10 to R12, R28 to R13, R1 to R14, R20 to R15, R12 to R16, R3 to R17, R29 to R18, R21 to R19, R25 to R2, R4 to R20, R13 to R21, R31 to R22, R15 to R24, R6 to R25, R30 to R26, R22 to R27, R14 to R28, R5 to R29, R17 to R3, R32 to R30, R24 to R31, R16 to R32, R7 to R33, R8 to R4, R9 to R5, R27 to R6, R19 to R7, R11 to R8, R2 to R9, RV2 to RV1, RV1 to RV2, SW22 to SW1, SW7 to SW10, SW9 to SW11, SW8 to SW12, SW10 to SW13, SW11 to SW14, SW12 to SW15, SW13 to SW16, SW14 to SW17, SW15 to SW18, SW17 to SW19, SW21 to SW2, SW16 to SW20, SW18 to SW21, SW19 to SW22, SW20 to SW23, SW35 to SW3, SW1 to SW4, SW2 to SW5, SW3 to SW6, SW4 to SW7, SW5 to SW8, SW6 to SW9
Other:
- board size 349.3 x 174.9 mm -> 168.5 x 353.4 mm

Commit message: Revert "Renumber some components"
This reverts commit 4c9a93e4336de2276d9b49e02718b6a92f997a6a.
Parts:
- moved J26 259.6 mm to (236.7, 129.4)
- moved J27 259.6 mm to (255.7, 79.3)
- moved J28 259.6 mm to (256.1, 129.4)
- moved J31 259.6 mm to (294.3, 79.3)
- moved J32 259.6 mm to (295.0, 129.4)
- moved J34 259.6 mm to (314.4, 129.4)
- moved J35 259.6 mm to (332.8, 79.3)
- moved J39 259.6 mm to (210.0, 89.3)
- moved J40 259.6 mm to (209.8, 139.3)
- moved J41 259.6 mm to (229.2, 89.3)
- moved J43 259.6 mm to (248.4, 89.3)
- moved J44 259.6 mm to (248.2, 139.3)
- moved J45 259.6 mm to (267.6, 89.3)
- moved J46 259.6 mm to (267.5, 139.3)
- moved J47 259.6 mm to (286.8, 89.3)
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- renumbered C1 to C2, C2 to C3, D2 to D1, D16 to D10, D17 to D11, D20 to D12, D22 to D13, D23 to D14, D26 to D15, D27 to D16, D32 to D17, D30 to D18, D34 to D19, D1 to D2, D36 to D20, D19 to D21, D29 to D22, D35 to D23, D10 to D24, D18 to D25, D25 to D26, D33 to D27, D6 to D28, D15 to D29, D24 to D30, D12 to D32, D5 to D33, D13 to D34, D21 to D35, D28 to D36, D8 to D5, D7 to D6, D9 to D7, D11 to D8, D14 to D9, J12 to J1, J14 to J11, J18 to J12, J5 to J13, J9 to J14, J13 to J15, J17 to J16, J4 to J17, J21 to J18, J1 to J19, J8 to J2, J2 to J20, J3 to J21, J39 to J24, J24 to J25, J40 to J26, J25 to J27, J41 to J28, J27 to J29, J16 to J3, J43 to J30, J26 to J31, J42 to J32, J28 to J33, J44 to J34, J29 to J35, J45 to J36, J30 to J37, J46 to J38, J31 to J39, J20 to J4, J47 to J40, J33 to J41, J49 to J42, J32 to J43, J48 to J44, J34 to J45, J50 to J46, J35 to J47, J51 to J48, J36 to J49, J7 to J5, J52 to J50, J38 to J51, J53 to J52, J37 to J53, J11 to J6, J15 to J7, J19 to J8, J6 to J9, R14 to R1, R12 to R10, R8 to R11, R16 to R12, R21 to R13, R28 to R14, R24 to R15, R32 to R16, R3 to R17, R11 to R18, R7 to R19, R9 to R2, R15 to R20, R19 to R21, R27 to R22, R31 to R24, R2 to R25, R10 to R26, R6 to R27, R13 to R28, R18 to R29, R17 to R3, R26 to R30, R22 to R31, R30 to R32, R1 to R33, R20 to R4, R29 to R5, R25 to R6, R33 to R7, R4 to R8, R5 to R9, RV2 to RV1, RV1 to RV2, SW4 to SW1, SW13 to SW10, SW14 to SW11, SW15 to SW12, SW16 to SW13, SW17 to SW14, SW18 to SW15, SW20 to SW16, SW19 to SW17, SW21 to SW18, SW22 to SW19, SW5 to SW2, SW23 to SW20, SW2 to SW21, SW1 to SW22, SW6 to SW3, SW3 to SW35, SW7 to SW4, SW8 to SW5, SW9 to SW6, SW10 to SW7, SW12 to SW8, SW11 to SW9
Other:
- board size 168.5 x 353.4 mm -> 349.3 x 174.9 mm

Commit message: Renumber some components
Parts:
- R18: renamed from R29; value 10K -> 1K
- R19: renamed from R21; value 10K -> 1K
- R2: renamed from R25; value 10K -> 1K
- R20: renamed from R4; value 10K -> 1K
- R21: renamed from R13; value 10K -> 1K
- R22: renamed from R31; value 10K -> 1K
- R23: value 10K -> 1K
- R24: renamed from R15; value 10K -> 1K
- R25: renamed from R6; value 10K -> 1K
- R3: renamed from R17; value 10K -> 1K
- R4: renamed from R8; value 10K -> 1K
- R5: renamed from R9; value 10K -> 1K
- R6: renamed from R27; value 10K -> 1K
- R7: renamed from R19; value 10K -> 1K
- R8: renamed from R11; value 10K -> 1K
- R9: renamed from R2; value 10K -> 1K
- moved J22 254.1 mm to (168.9, 201.6)
- moved J24 254.1 mm to (24.9, 263.4)
- moved J26 254.1 mm to (44.1, 263.4)
- moved J27 254.1 mm to (63.3, 263.4)
- moved J28 254.1 mm to (82.5, 263.4)
- moved J29 254.1 mm to (70.7, 253.4)
- moved J31 254.1 mm to (109.2, 253.4)
- moved J32 254.1 mm to (101.7, 263.4)
- moved J33 254.1 mm to (120.9, 263.4)
- moved J35 254.1 mm to (159.4, 263.4)
- moved J36 254.1 mm to (140.2, 263.4)
- moved J37 254.1 mm to (147.7, 253.4)
- moved J39 254.1 mm to (24.7, 313.5)
- moved J42 254.1 mm to (51.6, 303.6)
- moved J43 254.1 mm to (63.2, 313.5)
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- renumbered C2 to C1, C3 to C2, D2 to D1, D7 to D10, D34 to D11, D32 to D12, D8 to D13, D29 to D14, D10 to D15, D9 to D16, D25 to D17, D11 to D18, D12 to D19, D1 to D2, D21 to D20, D35 to D21, D30 to D22, D13 to D23, D14 to D24, D26 to D25, D15 to D26, D16 to D27, D22 to D28, D36 to D29, D18 to D30, D17 to D32, D27 to D33, D19 to D34, D20 to D35, D23 to D36, D33 to D5, D28 to D6, D5 to D7, D6 to D8, D24 to D9, J19 to J1, J6 to J11, J1 to J12, J15 to J13, J11 to J14, J7 to J15, J3 to J17, J12 to J18, J8 to J19, J20 to J2, J4 to J20, J18 to J21, J39 to J24, J41 to J26, J43 to J27, J45 to J28, J27 to J29, J21 to J3, J29 to J30, J47 to J32, J49 to J33, J33 to J34, J53 to J35, J51 to J36, J35 to J37, J37 to J38, J40 to J39, J17 to J4, J24 to J40, J42 to J41, J26 to J42, J44 to J43, J28 to J44, J46 to J45, J48 to J46, J32 to J47, J30 to J48, J34 to J49, J13 to J5, J36 to J51, J54 to J52, J52 to J53, J38 to J54, J9 to J6, J5 to J7, J14 to J8, J2 to J9, R33 to R1, R26 to R10, R18 to R11, R10 to R12, R1 to R13, R28 to R14, R20 to R15, R12 to R16, R3 to R17, R30 to R26, R22 to R27, R14 to R28, R5 to R29, R32 to R30, R24 to R31, R16 to R32, R7 to R33, RV2 to RV1, RV1 to RV2, SW22 to SW1, SW7 to SW10, SW8 to SW11, SW9 to SW12, SW10 to SW13, SW11 to SW14, SW12 to SW15, SW13 to SW16, SW14 to SW17, SW15 to SW18, SW16 to SW19, SW21 to SW2, SW17 to SW20, SW18 to SW21, SW19 to SW22, SW20 to SW23, SW35 to SW3, SW1 to SW4, SW2 to SW5, SW3 to SW6, SW4 to SW7, SW5 to SW8, SW6 to SW9
Other:
- board size 349.3 x 174.9 mm -> 168.4 x 345.6 mm
