File: arduino-delay/arduino-delay.kicad_sch (KiCad schematic)
At the start: 42 parts, among them J1 Output, J2 CV, J3 Power, J4 Power, J9 Input, SW1 A, SW2 B, SW3 C, U2 TL074

Commit message: Arduino delay progress
Parts:
- added J10: Input, modular2:banana-jack, symbol Connector:Conn_01x01_Pin
- added J5: Conn_01x03_Socket, Connector_PinSocket_2.54mm:PinSocket_1x03_P2.54mm_Vertical, symbol Connector:Conn_01x03_Socket
- added J6: Conn_01x03_Pin, Connector_PinHeader_2.54mm:PinHeader_1x03_P2.54mm_Vertical, symbol Connector:Conn_01x03_Pin
- added J7: Output, modular2:banana-jack, symbol Connector:Conn_01x01_Pin
- added J8: CV, modular2:banana-jack, symbol Connector:Conn_01x01_Pin
Connections:
- net at C3.1, J9.1 (Pin_1): now also J5.1 (Pin_1)
- net at J2.1 (Pin_1), R12.2: now also J5.2 (Pin_2)
- net at J1.1 (Pin_1), R11.1: now also J5.3 (Pin_3)
- new net: J10.1 (Pin_1), J6.1 (Pin_1)
- new net: J6.2 (Pin_2), J8.1 (Pin_1)
- new net: J6.3 (Pin_3), J7.1 (Pin_1)

Commit message: Complete arduino delay
Parts:
- renumbered A2 to A1, C7 to C1, C1 to C2, C5 to C3, C6 to C5, C3 to C6, C2 to C7, J3 to J1, J8 to J10, J4 to J2, J9 to J3, J2 to J4, J1 to J6, J10 to J8, J6 to J9, R8 to R1, R7 to R10, R12 to R11, R13 to R12, R11 to R13, R6 to R2, R10 to R3, R3 to R4, R4 to R6, R9 to R7, R1 to R8, R2 to R9, RV8 to RV1, RV7 to RV2, RV1 to RV3, RV3 to RV5, RV9 to RV6, RV2 to RV7, RV5 to RV8, RV6 to RV9, SW3 to SW2, SW2 to SW3, U4 to U1

Commit message: Update audio mixer to new format
Parts:
- RV1, RV2, RV3, RV4, RV5, RV6, RV7, RV8, RV9: footprint Potentiometer_THT:Potentiometer_Alps_RK09K_Single_Vertical -> modular2:Potentiometer_Alps_RK09K_Single_Vertical - knob padding
Changed lines of the file:
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@@
 			)
 		)
-		(property "Footprint" "Potentiometer_THT:Potentiometer_Alps_RK09K_Single_Vertical"
+		(property "Footprint" "modular2:Potentiometer_Alps_RK09K_Single_Vertical - knob padding"
 			(at 34.29 43.18 0)
 			(effects
@@
 			)
 		)
-		(property "Footprint" "Potentiometer_THT:Potentiometer_Alps_RK09K_Single_Vertical"
+		(property "Footprint" "modular2:Potentiometer_Alps_RK09K_Single_Vertical - knob padding"
 			(at 119.38 172.72 0)
 			(effects
@@
 			)
 		)
-		(property "Footprint" "Potentiometer_THT:Potentiometer_Alps_RK09K_Single_Vertical"
+		(property "Footprint" "modular2:Potentiometer_Alps_RK09K_Single_Vertical - knob padding"
 			(at 133.35 105.41 0)
 			(effects
@@
 			)
 		)
-		(property "Footprint" "Potentiometer_THT:Potentiometer_Alps_RK09K_Single_Vertical"
+		(property "Footprint" "modular2:Potentiometer_Alps_RK09K_Single_Vertical - knob padding"
 			(at 106.68 130.81 0)
 			(effects
@@
 			)
 		)
-		(property "Footprint" "Potentiometer_THT:Potentiometer_Alps_RK09K_Single_Vertical"
+		(property "Footprint" "modular2:Potentiometer_Alps_RK09K_Single_Vertical - knob padding"
 			(at 151.13 160.02 0)
 			(effects
@@
 			)
 		)
-		(property "Footprint" "Potentiometer_THT:Potentiometer_Alps_RK09K_Single_Vertical"
+		(property "Footprint" "modular2:Potentiometer_Alps_RK09K_Single_Vertical - knob padding"
 			(at 35.56 92.71 0)
 			(effects
@@
 			)
 		)
-		(property "Footprint" "Potentiometer_THT:Potentiometer_Alps_RK09K_Single_Vertical"
+		(property "Footprint" "modular2:Potentiometer_Alps_RK09K_Single_Vertical - knob padding"
 			(at 34.29 58.42 0)
 			(effects
@@
 			)
 		)
-		(property "Footprint" "Potentiometer_THT:Potentiometer_Alps_RK09K_Single_Vertical"
+		(property "Footprint" "modular2:Potentiometer_Alps_RK09K_Single_Vertical - knob padding"
 			(at 39.37 133.35 0)
 			(effects
@@
 			)
 		)
-		(property "Footprint" "Potentiometer_THT:Potentiometer_Alps_RK09K_Single_Vertical"
+		(property "Footprint" "modular2:Potentiometer_Alps_RK09K_Single_Vertical - knob padding"
 			(at 35.56 76.2 0)
 			(effects
