File: arduino-delay/arduino-delay.kicad_sch (KiCad schematic)
At the start: 47 parts, among them J1 Power, J10 CV, J2 Power, J3 Input, J4 CV, J5 Conn_01x03_Socket, J6 Output, J7 Output, J8 Input, J9 Conn_01x03_Pin, SW1 A, SW2 C, SW3 B, U2 TL074

Commit message: Update some pdfs
Parts:
- U1: value ~ -> (none)
