File: arduino-delay/arduino-delay.kicad_pcb (KiCad board)
At the start: 2 copper layers, 55.1 x 156.5 mm, 48 parts, among them J1 Output, J2 CV, J3 Power, J4 Power, J9 Input, SW1 A, SW2 B, SW3 C, U2 TL074

Commit message: Arduino delay progress
Parts:
- added J10: Input, modular2:banana-jack, F.Cu at (97.3, 166.5)
- added J5: Conn_01x03_Socket, Connector_PinSocket_2.54mm:PinSocket_1x03_P2.54mm_Vertical, F.Cu at (51.3, 176.5)
- added J6: Conn_01x03_Pin, Connector_PinHeader_2.54mm:PinHeader_1x03_P2.54mm_Vertical, F.Cu at (113.0, 176.5)
- added J7: Output, modular2:banana-jack, F.Cu at (133.9, 166.5)
- added J8: CV, modular2:banana-jack, F.Cu at (115.7, 166.5)
- added REF**: MountingHole_3.2mm_M3, MountingHole:MountingHole_3.2mm_M3, F.Cu at (97.2, 90.5)
- added REF**: MountingHole_3.2mm_M3, MountingHole:MountingHole_3.2mm_M3, F.Cu at (133.8, 90.5)
- added REF**: MountingHole_3.2mm_M3, MountingHole:MountingHole_3.2mm_M3, F.Cu at (97.2, 44.5)
- added REF**: MountingHole_3.2mm_M3, MountingHole:MountingHole_3.2mm_M3, F.Cu at (97.2, 176.5)
- added REF**: MountingHole_3.2mm_M3, MountingHole:MountingHole_3.2mm_M3, F.Cu at (133.8, 176.5)
- added REF**: MountingHole_3.2mm_M3, MountingHole:MountingHole_3.2mm_M3, F.Cu at (133.8, 44.5)
- moved J3 45.9 mm to (37.6, 35.5)
- moved RV4 42.2 mm to (33.0, 130.1)
- moved J1 42.1 mm to (72.1, 166.5)
- moved REF** 42.1 mm to (72.1, 44.5)
- moved REF** 42.1 mm to (72.1, 176.5)
- moved REF** 42.1 mm to (72.1, 90.5)
- moved RV1 42.1 mm to (69.6, 107.8)
- moved RV6 42.1 mm to (69.6, 152.5)
- moved RV7 42.1 mm to (69.6, 85.4)
- moved RV8 42.1 mm to (69.6, 63.0)
- moved J2 42.1 mm to (53.9, 166.5)
- moved RV5 42.1 mm to (51.4, 152.5)
- moved SW2 42.1 mm to (44.6, 102.0)
- moved A2 42.1 mm to (61.5, 82.5)
- moved C1 42.1 mm to (31.0, 75.5)
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Routing:
- net Net-(J5-Pin_1): track 94.5 -> 114.4 mm
- net Net-(J10-Pin_1): track 0.00 -> 19.9 mm
- net Net-(J6-Pin_3): track 0.00 -> 19.9 mm
- net Net-(J1-Pin_1): track 78.6 -> 98.5 mm
- net 5V: track 207.0 -> 187.4 mm
- net GND: track 441.0 -> 427.1 mm
- net Net-(J2-Pin_1): track 96.2 -> 106.2 mm
- net Net-(J6-Pin_2): track 0.00 -> 9.99 mm
- net 12V: track 85.2 -> 92.2 mm
- net -12V: track 84.4 -> 88.1 mm
- net Net-(A2-AREF): track 5.37 -> 4.61 mm
Other:
- board size 55.1 x 156.5 mm -> 116.9 x 151.8 mm
- board text added: "ARDUINO DELAY V1"

Commit message: Complete arduino delay
Parts:
- moved J10 7.13 mm to (122.8, 166.6)
- moved J7 7.13 mm to (141.0, 166.5)
- moved J8 7.13 mm to (104.4, 166.6)
- moved J9 7.13 mm to (120.2, 176.5)
- moved REF** 7.13 mm to (104.4, 90.5)
- moved REF** 7.13 mm to (141.0, 90.5)
- moved REF** 7.13 mm to (104.4, 44.5)
- moved REF** 7.13 mm to (104.4, 176.5)
- moved REF** 7.13 mm to (141.0, 176.5)
- moved REF** 7.13 mm to (141.0, 44.5)
- renumbered A2 to A1, C7 to C1, C1 to C2, C5 to C3, C6 to C5, C3 to C6, C2 to C7, J3 to J1, J8 to J10, J4 to J2, J9 to J3, J2 to J4, J1 to J6, J10 to J8, J6 to J9, R8 to R1, R7 to R10, R12 to R11, R13 to R12, R11 to R13, R6 to R2, R10 to R3, R3 to R4, R4 to R6, R9 to R7, R1 to R8, R2 to R9, RV8 to RV1, RV7 to RV2, RV1 to RV3, RV3 to RV5, RV9 to RV6, RV2 to RV7, RV5 to RV8, RV6 to RV9, SW3 to SW2, SW2 to SW3, U4 to U1
Other:
- board size 116.9 x 151.8 mm -> 124 x 151.8 mm

Commit message: Update audio mixer to new format
Parts:
- RV1, RV2, RV3, RV4, RV5, RV6, RV7, RV8, RV9: footprint Potentiometer_THT:Potentiometer_Alps_RK09K_Single_Vertical -> modular2:Potentiometer_Alps_RK09K_Single_Vertical - knob padding

Commit message: Update some designs
Parts:
- moved J10 6.50 mm to (117.0, 163.5)
- moved J7 6.50 mm to (135.2, 163.5)
- moved J8 6.50 mm to (98.6, 163.5)
- moved J9 6.50 mm to (114.4, 173.5)
- moved REF** 6.50 mm to (98.6, 87.5)
- moved REF** 6.50 mm to (98.6, 41.5)
- moved REF** 6.50 mm to (98.6, 173.5)
- moved REF** 6.50 mm to (135.2, 87.5)
- moved REF** 6.50 mm to (135.2, 173.5)
- moved REF** 6.50 mm to (135.2, 41.5)
- moved A1 0.87 mm to (60.6, 82.5)
- moved C1 0.87 mm to (42.2, 44.5)
- moved C3 0.87 mm to (44.1, 88.0)
- moved C4 0.87 mm to (62.1, 88.0)
- moved C5 0.87 mm to (37.6, 75.5)
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Other:
- board size 124 x 151.8 mm -> 119.1 x 151.8 mm
