File: arduino-delay/arduino-delay.kicad_pcb (KiCad board)
At the start: 2 copper layers, 119.1 x 151.8 mm, 59 parts, among them J1 Power, J10 CV, J2 Power, J3 Input, J4 CV, J5 Conn_01x03_Socket, J6 Output, J7 Output, J8 Input, J9 Conn_01x03_Pin, SW1 A, SW2 C, SW3 B, U2 TL074

Commit message: Update some gerbers
Parts:
- moved J2 4.72 mm to (68.7, 36.0)
- moved J1 4.72 mm to (32.1, 36.0)
Routing:
- net 5V: track 187.4 -> 213.3 mm
- net -12V: track 88.1 -> 114.0 mm
- net GND: track 427.1 -> 406.4 mm
- net 12V: track 92.2 -> 98.8 mm
