File: audio-mixer/audio-mixer.kicad_pcb (KiCad board)
At the start: 2 copper layers, 190 x 124.5 mm, 72 parts, among them J1 Input A1, J10 Output A, J11 Output B, J12 Conn_01x11_Socket, J13 AudioJack4, J14 Input A1, J15 Input B1, J16 Input A2, J17 Input B2, J18 Input A3, J19 Input B3, J2 Power, J20 Output A, J21 Output B, J22 Conn_01x11_Pin, J23 Conn_01x03_Pin, J3 Power, J4 Power, J5 Input B1, J6 Input A2, J7 Input B2, J8 Input A3, J9 Input B3, SW1 Iso A1, SW2 Iso B1, SW3 Iso A2, SW4 Iso B2, SW5 Iso A3, SW6 Iso B3, SW7 Iso A, SW8 Iso B, SW9 Mono/Stereo, U1 TL074

Commit message: Update some designs
Parts:
- added REF**: MountingHole_3.2mm_M3, MountingHole:MountingHole_3.2mm_M3, F.Cu at (104.9, 85.5)
- added REF**: MountingHole_3.2mm_M3, MountingHole:MountingHole_3.2mm_M3, F.Cu at (30.6, 220.5)
- added REF**: MountingHole_3.2mm_M3, MountingHole:MountingHole_3.2mm_M3, F.Cu at (32.2, 85.5)
- added REF**: MountingHole_3.2mm_M3, MountingHole:MountingHole_3.2mm_M3, F.Cu at (103.4, 220.5)
- moved J14 169.3 mm to (30.7, 189.2)
- moved J15 169.3 mm to (103.3, 189.2)
- moved J16 169.3 mm to (30.6, 210.0)
- moved J17 169.3 mm to (103.3, 210.0)
- moved J19 169.3 mm to (103.3, 230.8)
- moved J20 169.3 mm to (30.5, 258.6)
- moved J18 169.3 mm to (30.5, 230.8)
- moved J21 169.3 mm to (103.3, 258.6)
- moved J22 169.3 mm to (80.3, 270.5)
- moved J23 169.3 mm to (66.0, 281.5)
- moved REF** 169.3 mm to (30.6, 179.0)
- moved REF** 169.3 mm to (103.3, 179.0)
- moved REF** 169.3 mm to (31.0, 284.0)
- moved REF** 169.3 mm to (103.7, 284.0)
- moved RV1 9.66 mm to (56.3, 61.8)
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Other:
- board size 190 x 124.5 mm -> 87.7 x 259.5 mm
