File: audio-mixer/audio-mixer.kicad_pcb (KiCad board)
At the start: 2 copper layers, 87.7 x 259.5 mm, 76 parts, among them J1 Input A1, J10 Output A, J11 Output B, J12 Conn_01x11_Socket, J13 AudioJack4, J14 Input A1, J15 Input B1, J16 Input A2, J17 Input B2, J18 Input A3, J19 Input B3, J2 Power, J20 Output A, J21 Output B, J22 Conn_01x11_Pin, J23 Conn_01x03_Pin, J3 Power, J4 Power, J5 Input B1, J6 Input A2, J7 Input B2, J8 Input A3, J9 Input B3, SW1 Iso A1, SW2 Iso B1, SW3 Iso A2, SW4 Iso B2, SW5 Iso A3, SW6 Iso B3, SW7 Iso A, SW8 Iso B, SW9 Mono/Stereo, U1 TL074

Commit message: Extra channels in audio mixer
Parts:
- added C10: 10uF, Capacitor_THT:C_Disc_D4.3mm_W1.9mm_P5.00mm, F.Cu at (31.2, 142.1)
- added C11: 10uF, Capacitor_THT:C_Disc_D4.3mm_W1.9mm_P5.00mm, F.Cu at (70.7, 118.6)
- added C12: 10uF, Capacitor_THT:C_Disc_D4.3mm_W1.9mm_P5.00mm, F.Cu at (90.9, 142.0)
- added C9: 10uF, Capacitor_THT:C_Disc_D4.3mm_W1.9mm_P5.00mm, F.Cu at (51.2, 118.9)
- added J24: Input A4, modular2:banana-jack, F.Cu at (24.5, 108.4)
- added J25: Input A5, modular2:banana-jack, F.Cu at (24.5, 129.2)
- added J26: Input A4, modular2:banana-jack, F.Cu at (152.6, 110.5)
- added J27: Input A5, modular2:banana-jack, F.Cu at (152.5, 131.3)
- added J28: Input B4, modular2:banana-jack, F.Cu at (225.4, 110.5)
- added J29: Input B5, modular2:banana-jack, F.Cu at (225.4, 131.3)
- added J30: Input B4, modular2:banana-jack, F.Cu at (97.3, 108.4)
- added J31: Input B5, modular2:banana-jack, F.Cu at (97.3, 129.2)
- added R15: 100K, Resistor_THT:R_Axial_DIN0207_L6.3mm_D2.5mm_P10.16mm_Horizontal, F.Cu at (46.1, 121.7)
- added R16: 100K, Resistor_THT:R_Axial_DIN0207_L6.3mm_D2.5mm_P10.16mm_Horizontal, F.Cu at (38.4, 142.1)
- added R17: 100K, Resistor_THT:R_Axial_DIN0207_L6.3mm_D2.5mm_P10.16mm_Horizontal, F.Cu at (75.7, 121.5)
- added R18: 100K, Resistor_THT:R_Axial_DIN0207_L6.3mm_D2.5mm_P10.16mm_Horizontal, F.Cu at (83.6, 142.0)
- added RV10: 100K - A5, modular2:Potentiometer_Alps_RK09K_Single_Vertical - knob padding, F.Cu at (48.7, 136.8)
- added RV11: 100K - B4, modular2:Potentiometer_Alps_RK09K_Single_Vertical - knob padding, F.Cu at (68.2, 116.0)
- added RV12: 100K - B5, modular2:Potentiometer_Alps_RK09K_Single_Vertical - knob padding, F.Cu at (68.2, 136.8)
- added RV9: 100K - A4, modular2:Potentiometer_Alps_RK09K_Single_Vertical - knob padding, F.Cu at (48.7, 116.0)
- added SW10: Iso A4, modular2:switch1, F.Cu at (36.4, 108.4)
- added SW11: Iso A5, modular2:switch1, F.Cu at (36.4, 129.2)
- added SW12: Iso B4, modular2:switch1, F.Cu at (85.6, 108.4)
- added SW13: Iso B5, modular2:switch1, F.Cu at (85.6, 129.2)
- J12: value Conn_01x11_Socket -> Conn_01x15_Socket; footprint Connector_PinSocket_2.54mm:PinSocket_1x11_P2.54mm_Vertical -> Connector_PinSocket_2.54mm:PinSocket_1x15_P2.54mm_Vertical
- J22: value Conn_01x11_Pin -> Conn_01x15_Pin; footprint Connector_PinHeader_2.54mm:PinHeader_1x11_P2.54mm_Vertical -> Connector_PinHeader_2.54mm:PinHeader_1x15_P2.54mm_Vertical
- moved J19 186.7 mm to (225.4, 89.6)
- moved J14 186.7 mm to (152.7, 48.0)
- moved J15 186.7 mm to (225.4, 48.0)
- moved J16 186.7 mm to (152.7, 68.8)
- moved J17 186.7 mm to (225.4, 68.8)
- moved REF** 186.7 mm to (152.7, 37.8)
- moved REF** 186.7 mm to (225.4, 37.8)
- moved J18 186.7 mm to (152.6, 89.6)
- moved REF** 171.4 mm to (225.3, 100.0)
- moved REF** 171.4 mm to (152.6, 100.0)
- moved J22 161.5 mm to (206.9, 170.2)
- moved J20 158.0 mm to (152.6, 158.3)
- moved J23 158.0 mm to (188.1, 181.2)
- moved J21 158.0 mm to (225.4, 158.3)
- moved REF** 158.0 mm to (153.1, 183.7)
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Connections:
- J12 pad 10: Net-(J12-Pin_10) -> Net-(J10-Pin_1)
- J12 pad 11: Net-(J1-Pin_1) -> Net-(J12-Pin_11)
- J12 pad 4: Net-(J11-Pin_1) -> Net-(J12-Pin_4)
- J12 pad 6: Net-(J12-Pin_6) -> Net-(J11-Pin_1)
- J12 pad 7: GND -> Net-(J12-Pin_7)
- J12 pad 8: Net-(J10-Pin_1) -> Net-(J12-Pin_8)
- J12 pad 9: Net-(J12-Pin_9) -> GND
- J13 pad R1: Net-(J12-Pin_6) -> Net-(J12-Pin_8)
- J13 pad T: Net-(J12-Pin_5) -> Net-(J12-Pin_7)
- J22 pad 10: Net-(J16-Pin_1) -> Net-(J20-Pin_1)
- J22 pad 11: Net-(J14-Pin_1) -> Net-(J22-Pin_11)
- J22 pad 4: Net-(J21-Pin_1) -> Net-(J22-Pin_4)
- J22 pad 6: Net-(J22-Pin_6) -> Net-(J21-Pin_1)
- J22 pad 8: Net-(J20-Pin_1) -> Net-(J22-Pin_8)
- J22 pad 9: Net-(J18-Pin_1) -> Net-(J22-Pin_9)
- J23 pad 1: Net-(J22-Pin_5) -> Net-(J22-Pin_7)
- J23 pad 2: Net-(J22-Pin_6) -> Net-(J22-Pin_8)
- J23 pad 3: Net-(J22-Pin_7) -> Net-(J22-Pin_9)
- J6 pad 1: Net-(J12-Pin_10) -> Net-(J12-Pin_14)
- J8 pad 1: Net-(J12-Pin_9) -> Net-(J12-Pin_13)
- R14 pad 2: Net-(J12-Pin_6) -> Net-(J12-Pin_8)
- R6 pad 2: Net-(J12-Pin_5) -> Net-(J12-Pin_7)
- SW3 pad 1: Net-(J12-Pin_10) -> Net-(J12-Pin_14)
- SW5 pad 1: Net-(J12-Pin_9) -> Net-(J12-Pin_13)
Routing:
- net GND: track 243.8 -> 418.7 mm
- net Net-(J12-Pin_14): track 0.00 -> 138.6 mm
- net Net-(J12-Pin_13): track 0.00 -> 119.7 mm
- net Net-(J12-Pin_10): track 101.9 -> 0.00 mm
- net Net-(J12-Pin_12): track 0.00 -> 100.7 mm
- net Net-(J12-Pin_4): track 0.00 -> 100.3 mm
- net Net-(J22-Pin_12): track 0.00 -> 87.0 mm
- net Net-(J22-Pin_4): track 0.00 -> 86.6 mm
- net Net-(J12-Pin_9): track 83.0 -> 0.00 mm
- net Net-(J12-Pin_11): track 0.00 -> 81.8 mm
- net Net-(J22-Pin_11): track 0.00 -> 68.0 mm
- net Net-(J22-Pin_5): track 12.8 -> 67.7 mm
- net Net-(J12-Pin_5): track 29.4 -> 81.3 mm
- net Net-(U1C--): track 75.6 -> 117.6 mm
- net Net-(U1D--): track 74.4 -> 115.6 mm
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Other:
- board size 87.7 x 259.5 mm -> 214.2 x 167.2 mm
