File: diode-ladder-filter/diode-ladder-filter.kicad_pcb (KiCad board)
At the start: 2 copper layers, 64.9 x 256.2 mm, 85 parts, among them J1 Power, J10 Input, J11 Output, J12 Conn_01x04_Pin, J2 Power, J3 CV1, J4 CV2, J5 Input, J6 Output, J7 Conn_01x04_Socket, J8 CV1, J9 CV2, SW1 Resonance_safety, SW2 LPF, SW3 HPF, SW4 BPF, U1 TL074, U2 TL074

Commit message: Update some designs
Parts:
- removed F0, F1, F2, F3: foot, modular2:foot
- moved H8 128.1 mm to (118.5, 154.3)
- moved H6 128.1 mm to (118.5, 47.0)
- moved H7 128.0 mm to (62.1, 154.3)
- moved H5 128.0 mm to (62.1, 47.0)
- moved J10 127.4 mm to (65.5, 138.3)
- moved J8 127.4 mm to (65.7, 77.3)
- moved J11 127.4 mm to (115.0, 138.4)
- moved J12 127.4 mm to (86.4, 156.3)
- moved J9 127.4 mm to (65.6, 97.3)
- moved H4 89.0 mm to (194.5, 152.5)
- moved H2 89.0 mm to (194.5, 45.2)
- moved C1 76.0 mm to (188.6, 86.0)
- moved C10 76.0 mm to (181.6, 120.6)
- moved C3 76.0 mm to (138.4, 112.2)
- moved D7 76.0 mm to (183.7, 95.9)
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Other:
- board size 64.9 x 256.2 mm -> 140.5 x 130.6 mm
- board text added: "DIODE LADDER FILTER V3"
- board text removed: "DIODE LADDER FILTER V2"
